File: OSC1.sch (EAGLE design)
At the start: 23 parts

Commit message: Board retraced
Parts:
- JP1: value STM32F3DISCO-LEFT -> STM32F3-DISCO LEFT; device pinhead:PINHD-2X20 -> pinhead:PINHD-2X19
Changed lines of the file:
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@@
 <part name="R18" library="rcl" deviceset="R-EU_" device="R1206" value="20K"/>
 <part name="GEN" library="wirepad" deviceset="2,54/0,8" device="" value="0-3V"/>
-<part name="JP1" library="pinhead" deviceset="PINHD-2X20" device="" value="STM32F3DISCO-LEFT"/>
+<part name="JP1" library="pinhead" deviceset="PINHD-2X19" device="" value="STM32F3-DISCO LEFT"/>
 </parts>
 <sheets>
@@
 <instance part="R18" gate="G$1" x="2.54" y="35.56"/>
 <instance part="GEN" gate="P" x="-12.7" y="35.56"/>
-<instance part="JP1" gate="A" x="99.06" y="139.7"/>
+<instance part="JP1" gate="G$1" x="99.06" y="142.24"/>
 </instances>
 <busses>
@@
 </segment>
 <segment>
-<pinref part="JP1" gate="A" pin="3"/>
 <pinref part="GND2" gate="1" pin="GND"/>
 <wire x1="96.52" y1="160.02" x2="71.12" y2="160.02" width="0.1524" layer="91"/>
 <wire x1="71.12" y1="160.02" x2="71.12" y2="157.48" width="0.1524" layer="91"/>
+<pinref part="JP1" gate="G$1" pin="3"/>
 </segment>
 </net>
@@
 </segment>
 <segment>
-<pinref part="JP1" gate="A" pin="33"/>
 <wire x1="96.52" y1="121.92" x2="76.2" y2="121.92" width="0.1524" layer="91"/>
 <label x="78.74" y="121.92" size="1.778" layer="95"/>
+<pinref part="JP1" gate="G$1" pin="33"/>
 </segment>
 </net>
@@
 </segment>
 <segment>
-<pinref part="JP1" gate="A" pin="22"/>
 <wire x1="124.46" y1="137.16" x2="104.14" y2="137.16" width="0.1524" layer="91"/>
 <label x="119.38" y="137.16" size="1.778" layer="95"/>
+<pinref part="JP1" gate="G$1" pin="22"/>
 </segment>
 </net>
@@
 </segment>
 <segment>
-<pinref part="JP1" gate="A" pin="23"/>
 <wire x1="96.52" y1="134.62" x2="76.2" y2="134.62" width="0.1524" layer="91"/>
 <label x="63.5" y="134.62" size="1.778" layer="95"/>
+<pinref part="JP1" gate="G$1" pin="23"/>
 </segment>
 </net>
@@
 </segment>
 <segment>
-<pinref part="JP1" gate="A" pin="8"/>
 <wire x1="124.46" y1="154.94" x2="104.14" y2="154.94" width="0.1524" layer="91"/>
 <label x="119.38" y="154.94" size="1.778" layer="95"/>
+<pinref part="JP1" gate="G$1" pin="8"/>
 </segment>
 </net>
 <net name="A1" class="0">
 <segment>
-<pinref part="JP1" gate="A" pin="9"/>
 <wire x1="96.52" y1="152.4" x2="76.2" y2="152.4" width="0.1524" layer="91"/>
 <label x="78.74" y="152.4" size="1.778" layer="95"/>
+<pinref part="JP1" gate="G$1" pin="9"/>
 </segment>
 <segment>
@@
 </segment>
 <segment>
-<pinref part="JP1" gate="A" pin="24"/>
 <wire x1="124.46" y1="134.62" x2="104.14" y2="134.62" width="0.1524" layer="91"/>
 <label x="119.38" y="134.62" size="1.778" layer="95"/>
+<pinref part="JP1" gate="G$1" pin="24"/>
 </segment>
 </net>
@@
 </segment>
 <segment>
-<pinref part="JP1" gate="A" pin="20"/>
 <wire x1="124.46" y1="139.7" x2="104.14" y2="139.7" width="0.1524" layer="91"/>
 <label x="119.38" y="139.7" size="1.778" layer="95"/>
+<pinref part="JP1" gate="G$1" pin="20"/>
 </segment>
 </net>
@@
 </segment>
 <segment>
-<pinref part="JP1" gate="A" pin="37"/>
 <wire x1="76.2" y1="116.84" x2="96.52" y2="116.84" width="0.1524" layer="91"/>
 <label x="78.74" y="116.84" size="1.778" layer="95"/>
+<pinref part="JP1" gate="G$1" pin="37"/>
 </segment>
 </net>
@@
 </segment>
 <segment>
-<pinref part="JP1" gate="A" pin="6"/>
 <wire x1="124.46" y1="157.48" x2="104.14" y2="157.48" width="0.1524" layer="91"/>
 <label x="119.38" y="157.48" size="1.778" layer="95"/>
+<pinref part="JP1" gate="G$1" pin="6"/>
 </segment>
 </net>
@@
 </segment>
 <segment>
-<pinref part="JP1" gate="A" pin="38"/>
 <wire x1="124.46" y1="116.84" x2="104.14" y2="116.84" width="0.1524" layer="91"/>
 <label x="119.38" y="116.84" size="1.778" layer="95"/>
+<pinref part="JP1" gate="G$1" pin="38"/>
 </segment>
 </net>
 <net name="DAC" class="0">
 <segment>
-<pinref part="JP1" gate="A" pin="16"/>
 <wire x1="124.46" y1="144.78" x2="104.14" y2="144.78" width="0.1524" layer="91"/>
 <label x="116.84" y="144.78" size="1.778" layer="95"/>
+<pinref part="JP1" gate="G$1" pin="16"/>
 </segment>
 <segment>
@@
 </segment>
 <segment>
-<pinref part="JP1" gate="A" pin="35"/>
 <wire x1="76.2" y1="119.38" x2="96.52" y2="119.38" width="0.1524" layer="91"/>
 <label x="78.74" y="119.38" size="1.778" layer="95"/>
+<pinref part="JP1" gate="G$1" pin="35"/>
 </segment>
 </net>
 <net name="B30" class="0">
 <segment>
-<pinref part="JP1" gate="A" pin="19"/>
 <wire x1="76.2" y1="139.7" x2="96.52" y2="139.7" width="0.1524" layer="91"/>
 <label x="78.74" y="139.7" size="1.778" layer="95"/>
+<pinref part="JP1" gate="G$1" pin="19"/>
 </segment>
 <segment>
@@
 </segment>
 <segment>
-<pinref part="JP1" gate="A" pin="5"/>
 <wire x1="76.2" y1="157.48" x2="96.52" y2="157.48" width="0.1524" layer="91"/>
 <label x="76.2" y="157.48" size="1.778" layer="95"/>
-</segment>
-</net>
+<pinref part="JP1" gate="G$1" pin="5"/>
+</segment>
+</net>
